Commit message: FIX SLAM.

File: clean_robot_ws/src/clean_robot_description/urdf/base.urdf.xacro (robot description, xacro)
@@ -10,5 +10,5 @@
     <visual>
       <geometry>
-        <box size="0.4 0.3 0.15"/>
+        <cylinder radius="0.045" length="0.08"/>
       </geometry>
       <material name="blue">

File: clean_robot_ws/src/clean_robot_description/urdf/clean_robot.urdf.xacro (robot description, xacro)
@@ -1,7 +1,54 @@
 <?xml version="1.0"?>
-<robot name="clean_robot"
-       xmlns:xacro="http://www.ros.org/wiki/xacro">
+<robot name="clean_robot" xmlns:xacro="http://www.ros.org/wiki/xacro">
     <xacro:include filename="base.urdf.xacro"/>
     <xacro:include filename="wheels.urdf.xacro"/>
     <xacro:include filename="sensors.urdf.xacro"/>
+    <webots>
+        <plugin type="clean_robot_simulation.my_robot_driver.MyRobotDriver" />
+        <device reference="rgb_camera" type="Camera">
+            <ros>
+                <topicName>/camera/image_raw</topicName>
+                <alwaysOn>true</alwaysOn>
+                <frameName>camera_link</frameName>
+                <alwaysOn>true</alwaysOn>
+            </ros>
+        </device>
+        <device reference="depth_camera" type="RangeFinder">
+        <ros>
+            <topicName>/depth_camera/image_depth</topicName>
+            <alwaysOn>true</alwaysOn>
+        </ros>
+        </device>
+        <device reference="lidar" type="Lidar">
+        <ros>
+            <topicName>/scan</topicName>
+            <alwaysOn>true</alwaysOn>
+            <frameName>lidar_link</frameName>
+            <alwaysOn>true</alwaysOn>
+            </ros>
+        </device>
+        <device reference="gps" type="GPS">
+            <ros>
+                <alwaysOn>true</alwaysOn>
+            </ros>
+        </device>
+        <device reference="inertial_unit" type="InertialUnit">
+            <ros>
+                <alwaysOn>true</alwaysOn>
+            </ros>
+        </device>
+    </webots>
+    <ros2_control name="WebotsControl" type="system">
+        <hardware>
+            <plugin>webots_ros2_control::Ros2ControlSystem</plugin>
+        </hardware>
+        <joint name="left_wheel_joint"> <command_interface name="velocity"/>
+            <state_interface name="position"/>
+            <state_interface name="velocity"/>
+        </joint>
+        <joint name="right_wheel_joint"> <command_interface name="velocity"/>
+            <state_interface name="position"/>
+            <state_interface name="velocity"/>
+        </joint>
+    </ros2_control>
 </robot>

File: clean_robot_ws/src/clean_robot_description/urdf/sensors.urdf.xacro (robot description, xacro)
@@ -4,13 +4,13 @@
     <parent link="base_link"/>
     <child link="lidar_link"/>
-    <origin xyz="0.1 0 0.1" rpy="0 0 0"/>
+    <origin xyz="0 0 0.0635" rpy="0 0 0"/>
   </joint>
   <link name="lidar_link">
     <visual>
       <geometry>
-        <cylinder radius="0.03" length="0.03"/>
+        <cylinder radius="0.025" length="0.015"/>
       </geometry>
-      <material name="red">
-        <color rgba="0.8 0.0 0.0 1.0"/>
+      <material name="black_lidar">
+        <color rgba="0.05 0.05 0.05 1.0"/>
       </material>
     </visual>
@@ -19,13 +19,13 @@
     <parent link="base_link"/>
     <child link="camera_link"/>
-    <origin xyz="0.2 0 0.05" rpy="0 0 0"/>
+    <origin xyz="0.055 0 0.0435" rpy="0 0.26 0"/>
   </joint>
   <link name="camera_link">
     <visual>
       <geometry>
-        <box size="0.02 0.05 0.02"/>
+        <box size="0.025 0.035 0.02"/>
       </geometry>
-      <material name="grey">
-        <color rgba="0.5 0.5 0.5 1.0"/>
+      <material name="dark_grey">
+        <color rgba="0.1 0.1 0.1 1.0"/>
       </material>
     </visual>

File: clean_robot_ws/src/clean_robot_description/urdf/wheels.urdf.xacro (robot description, xacro)
@@ -4,5 +4,5 @@
     <parent link="base_link"/>
     <child link="left_wheel_link"/>
-    <origin xyz="0.1 0.175 -0.05" rpy="-1.5708 0 0"/>
+    <origin xyz="0 0.045 -0.015" rpy="-1.5708 0 0"/>
     <axis xyz="0 0 1"/>
   </joint>
@@ -10,5 +10,5 @@
     <visual>
       <geometry>
-        <cylinder radius="0.05" length="0.04"/>
+        <cylinder radius="0.025" length="0.01"/>
       </geometry>
       <material name="black">
@@ -20,5 +20,5 @@
     <parent link="base_link"/>
     <child link="right_wheel_link"/>
-    <origin xyz="0.1 -0.175 -0.05" rpy="-1.5708 0 0"/>
+    <origin xyz="0 -0.045 -0.015" rpy="-1.5708 0 0"/>
     <axis xyz="0 0 1"/>
   </joint>
@@ -26,5 +26,5 @@
     <visual>
       <geometry>
-        <cylinder radius="0.05" length="0.04"/>
+        <cylinder radius="0.025" length="0.01"/>
       </geometry>
       <material name="black"/>
